Commit message: Fix lidar rotation

File: urdf/components/lidar.xacro (robot description, xacro)
@@ -29,5 +29,5 @@
       <parent link="${parent}"/>
       <child link="laser"/>
-      <origin xyz="${x} ${y} ${z}" rpy="0 0 0"/>
+      <origin xyz="${x} ${y} ${z}" rpy="0 0 ${pi}"/>
     </joint>
   </xacro:macro>
