Commit message: fix(moveit): mock hardware arg + fix S4 as fixed joint for 4-DOF arm
- jetank_ros2_control.urdf.xacro: add `hardware` arg (mock|serial, default
  mock) and pass it to the ros2_control macro, so MoveIt can drive the arm
  in software with no motors connected.
- components/arm.xacro: make S4_joint fixed. Servo 4 is repurposed for the
  gripper, so the wrist pitch is not actuated; modelling it fixed keeps the
  'arm' planning chain a clean 4-DOF (S1,S2,S3,S5) group that matches
  ros2_control, the arm_controller, and the SRDF named poses.

Part of feature/moveit-mock-arm (MoveIt mock loop). See companion commits
in jetank_motor_control and jetank_moveit_config.

Co-Authored-By: Claude Opus 4.8 (1M context) <noreply@anthropic.com>

File: urdf/components/arm.xacro (robot description, xacro)
@@ -130,12 +130,12 @@
       </inertial>
     </link>
-    <!-- S4 Joint - Wrist pitch (maps to Servo ID 4) -->
-    <joint name="S4_joint" type="revolute">
+    <!-- S4 Joint - Wrist pitch. FIXED: Servo ID 4 is repurposed to drive the
+         gripper, so the wrist pitch is not actuated. Modelling it as fixed
+         keeps the 'arm' planning chain a clean 4-DOF (S1, S2, S3, S5) group
+         that matches ros2_control, the arm_controller, and the SRDF poses. -->
+    <joint name="S4_joint" type="fixed">
       <origin xyz="0.09 0 0" rpy="0 0 0"/>
       <parent link="S3_link"/>
       <child link="S4_link"/>
-      <axis xyz="0 1 0"/>
-      <limit lower="-1.57" upper="1.57" effort="0.5" velocity="1.57"/>
-      <dynamics damping="0.05" friction="0.05"/>
     </joint>
     <link name="S4_link">

File: urdf/jetank_ros2_control.urdf.xacro (robot description, xacro)
@@ -5,4 +5,7 @@
   <xacro:arg name="use_sim" default="false"/>
   <xacro:arg name="use_ros2_control" default="true"/>
+  <!-- hardware backend when use_sim is false: mock | serial (default mock,
+       so MoveIt can drive the arm in software with no motors connected). -->
+  <xacro:arg name="hardware" default="mock"/>
   <!-- Import component macros -->
   <xacro:include filename="$(find jetank_description)/urdf/components/arm.xacro"/>
@@ -56,5 +59,5 @@
   <!-- ros2_control (conditional) -->
   <xacro:if value="$(arg use_ros2_control)">
-    <xacro:jetank_ros2_control use_sim="$(arg use_sim)"/>
+    <xacro:jetank_ros2_control use_sim="$(arg use_sim)" hardware="$(arg hardware)"/>
   </xacro:if>
   <!-- Gazebo properties -->

Commit message: fix(arm): make S4_joint fixed (4-DOF arm, no free/uncontrolled joint)
Servo 4 is repurposed to drive the gripper, so S4 has no ros2_control
interface. As a revolute joint it was an uncontrolled DOF: it drooped under
gravity in Gazebo and left MoveIt without state/controller for it ("complete
state of the robot is not yet known. Missing S4_joint"). Fixing it makes the
arm a clean 4-DOF chain (S1,S2,S3,S5), matching the SRDF/controller intent.

Co-Authored-By: Claude Opus 4.8 (1M context) <noreply@anthropic.com>

File: urdf/components/arm.xacro (robot description, xacro)
@@ -130,12 +130,13 @@
       </inertial>
     </link>
-    <!-- S4 Joint - Wrist pitch (maps to Servo ID 4) -->
-    <joint name="S4_joint" type="revolute">
+    <!-- S4 Joint - Wrist pitch. Servo 4 is repurposed to drive the gripper, so
+         S4 is NOT an actuated arm joint: it has no ros2_control interface. It is
+         therefore FIXED so the arm is a clean 4-DOF chain (S1,S2,S3,S5). Leaving
+         it revolute makes it an uncontrolled free joint (droops in Gazebo) and
+         adds a DOF MoveIt has no state/controller for. -->
+    <joint name="S4_joint" type="fixed">
       <origin xyz="0.09 0 0" rpy="0 0 0"/>
       <parent link="S3_link"/>
       <child link="S4_link"/>
-      <axis xyz="0 1 0"/>
-      <limit lower="-1.57" upper="1.57" effort="0.5" velocity="1.57"/>
-      <dynamics damping="0.05" friction="0.05"/>
     </joint>
     <link name="S4_link">

Commit message: feat(arm): widen S3 elbow limit to +/-2.356 rad (270deg real servo travel)
S3 was capped at +/-1.57 (180deg) but the real servo travels ~270deg centred
on forearm-colinear. Widening lets the elbow fold down ~8cm lower for low reach.

Co-Authored-By: Claude Opus 4.8 (1M context) <noreply@anthropic.com>

File: urdf/components/arm.xacro (robot description, xacro)
@@ -100,4 +100,7 @@
     </link>
     <!-- S3 Joint - Elbow pitch (maps to Servo ID 3) -->
+    <!-- Real servo travel ~270 deg, centred on forearm colinear with upper arm
+         (S3=0). Limits +/-135 deg (+/-2.356 rad) so the elbow can fold the
+         forearm down far enough to reach low/floor targets. -->
     <joint name="S3_joint" type="revolute">
       <origin xyz="0.11 0 0" rpy="0 1.5708 0"/>
@@ -105,5 +108,5 @@
       <child link="S3_link"/>
       <axis xyz="0 1 0"/>
-      <limit lower="-1.57" upper="1.57" effort="1.0" velocity="1.57"/>
+      <limit lower="-2.356" upper="2.356" effort="1.0" velocity="1.57"/>
       <dynamics damping="0.1" friction="0.1"/>
     </joint>

Commit message: feat(arm): extend S2 forward limit to +2.356 (45deg past horizontal)
Lets the upper arm point forward-and-down for low reach. +S2 forward.

Co-Authored-By: Claude Opus 4.8 (1M context) <noreply@anthropic.com>

File: urdf/components/arm.xacro (robot description, xacro)
@@ -69,4 +69,7 @@
     </link>
     <!-- S2 Joint - Shoulder pitch (maps to Servo ID 2) -->
+    <!-- S2=0 points the upper arm UP. +S2 swings it forward. Upper limit raised
+         to +2.356 (135deg) so it can rotate ~45deg PAST horizontal-forward,
+         pointing the upper arm forward-and-down for low/floor reach. -->
     <joint name="S2_joint" type="revolute">
       <origin xyz="0.0075 0 0.0275" rpy="0 -1.5708 0"/>
@@ -74,5 +77,5 @@
       <child link="S2_link"/>
       <axis xyz="0 1 0"/>
-      <limit lower="-1.57" upper="1.57" effort="1.0" velocity="1.57"/>
+      <limit lower="-1.57" upper="2.356" effort="1.0" velocity="1.57"/>
       <dynamics damping="0.1" friction="0.1"/>
     </joint>
