Commit message: fix(gripper): raise effort to 5N, remove URDF mimic tag, reduce damping/friction
Remove the URDF <mimic> tag from gripper_right_joint — the ros2_control
resource manager's native mimic (param name="mimic" in ros2_control.xacro)
handles mirroring without creating a Gazebo physics constraint that fights
the GripperActionController's position commands.

Raise effort limit from 0.5 N to 5 N to match the GripperActionController
max_effort setting. Lower joint damping (0.1->0.01) and friction (0.05->0.0)
so the position controller's low-gain (kp=0.1 in ign_ros2_control Fortress)
can slide the finger without stalling. Reduce contact stiffness kp on finger
links from 1e6 to 1e4 for the same reason. Raise velocity limit to 0.5 m/s.

Verified in Gazebo Fortress: gripper_left_joint reaches 0.04 (open) and
returns to ~0.0 (closed); gripper_right_joint_mimic mirrors correctly.

Co-Authored-By: Claude Opus 4.8 (1M context) <noreply@anthropic.com>

File: urdf/components/gripper.xacro (robot description, xacro)
@@ -37,6 +37,8 @@
       <child link="gripper_left_link"/>
       <axis xyz="0 1 0"/>
-      <limit lower="0.0" upper="0.04" effort="0.5" velocity="0.1"/>
-      <dynamics damping="0.1" friction="0.05"/>
+      <!-- effort raised to 5 N (was 0.5) so GripperActionController can overcome
+           damping without stalling -->
+      <limit lower="0.0" upper="0.04" effort="5.0" velocity="0.5"/>
+      <dynamics damping="0.01" friction="0.0"/>
     </joint>
     <link name="gripper_left_link">
@@ -62,5 +64,10 @@
       </inertial>
     </link>
-    <!-- Right finger (mirrored) -->
+    <!-- Right finger (mirrored).
+         The URDF <mimic> tag is intentionally REMOVED here. The ros2_control
+         resource manager's native mimic mechanism (param name="mimic" in
+         ros2_control.xacro) mirrors gripper_right to gripper_left without
+         creating a Gazebo physics mimic constraint that would oppose the
+         GripperActionController's position commands. -->
     <joint name="gripper_right_joint" type="prismatic">
       <origin xyz="0 -0.04 0" rpy="0 0 0"/>
@@ -68,7 +75,7 @@
       <child link="gripper_right_link"/>
       <axis xyz="0 -1 0"/>
-      <limit lower="0.0" upper="0.04" effort="0.5" velocity="0.1"/>
-      <dynamics damping="0.1" friction="0.05"/>
-      <mimic joint="gripper_left_joint" multiplier="1.0" offset="0"/>
+      <!-- effort raised to 5 N (was 0.5) — consistent with left finger -->
+      <limit lower="0.0" upper="0.04" effort="5.0" velocity="0.5"/>
+      <dynamics damping="0.01" friction="0.0"/>
     </joint>
     <link name="gripper_right_link">
@@ -100,15 +107,19 @@
     <gazebo reference="gripper_left_link">
       <material>Gazebo/DarkGrey</material>
-      <kp>1000000.0</kp>
-      <kd>100.0</kd>
-      <mu1>1.0</mu1>
-      <mu2>1.0</mu2>
+      <!-- Reduced contact stiffness from 1e6 to 1e4 so the joint is not
+           fighting a rigid contact force at rest. Friction also reduced
+           so the low-gain position controller (kp=0.1 in ign_ros2_control
+           Fortress) can slide the finger without stalling. -->
+      <kp>10000.0</kp>
+      <kd>10.0</kd>
+      <mu1>0.5</mu1>
+      <mu2>0.5</mu2>
     </gazebo>
     <gazebo reference="gripper_right_link">
       <material>Gazebo/DarkGrey</material>
-      <kp>1000000.0</kp>
-      <kd>100.0</kd>
-      <mu1>1.0</mu1>
-      <mu2>1.0</mu2>
+      <kp>10000.0</kp>
+      <kd>10.0</kd>
+      <mu1>0.5</mu1>
+      <mu2>0.5</mu2>
     </gazebo>
   </xacro:macro>

Commit message: fix(gripper): restore URDF <mimic> tag for robot_state_publisher TF
Restores `<mimic joint="gripper_left_joint" multiplier="1.0">` on
gripper_right_joint so robot_state_publisher can compute the
gripper_right_link transform from the kinematic model.

The prior fix removed this tag to avoid a Gazebo physics constraint that
stalled the joint; now the right finger is driven physically by a
separate ForwardCommandController + gripper_mimic_relay node (see
jetank_motor_control and jetank_ros_main changes), so the URDF mimic
is only used by RSP for TF and by MoveIt for joint-model correctness.

Co-Authored-By: Claude Opus 4.8 (1M context) <noreply@anthropic.com>

File: urdf/components/gripper.xacro (robot description, xacro)
@@ -65,9 +65,16 @@
     </link>
     <!-- Right finger (mirrored).
-         The URDF <mimic> tag is intentionally REMOVED here. The ros2_control
-         resource manager's native mimic mechanism (param name="mimic" in
-         ros2_control.xacro) mirrors gripper_right to gripper_left without
-         creating a Gazebo physics mimic constraint that would oppose the
-         GripperActionController's position commands. -->
+         URDF <mimic> tag RESTORED: robot_state_publisher reads this to compute
+         gripper_right_link TF and MoveIt needs the real URDF joint model.
+         The ros2_control native mimic params (<param name="mimic">) are REMOVED
+         from ros2_control.xacro because gz_ros2_control appends "_mimic" to the
+         published state interface name, producing "gripper_right_joint_mimic" in
+         /joint_states instead of the real URDF name "gripper_right_joint".
+         Physics: Gazebo Fortress may or may not enforce the URDF <mimic>
+         constraint. If it does (with effort=5 N this is plausible), both fingers
+         move together. If not, the right finger stays at 0 in physics but RSP
+         still shows the correct TF (mirrored from left joint via the URDF mimic).
+         Either way /joint_states carries "gripper_right_joint" (not _mimic) and
+         MoveIt's joint-not-found spam is eliminated. -->
     <joint name="gripper_right_joint" type="prismatic">
       <origin xyz="0 -0.04 0" rpy="0 0 0"/>
@@ -78,4 +85,5 @@
       <limit lower="0.0" upper="0.04" effort="5.0" velocity="0.5"/>
       <dynamics damping="0.01" friction="0.0"/>
+      <mimic joint="gripper_left_joint" multiplier="1.0" offset="0"/>
     </joint>
     <link name="gripper_right_link">

Commit message: fix(gripper): tighten finger origins +/-0.04 -> +/-0.018 so close grips
At q=0 the finger plates sat ~5 cm apart, so 'closed' never looked closed and
the grab appeared to only open. Origins now place the plates ~6 mm apart when
closed (q=0) and ~11 cm open (q=0.04); both fingers come together visibly.

Co-Authored-By: Claude Opus 4.8 (1M context) <noreply@anthropic.com>

File: urdf/components/gripper.xacro (robot description, xacro)
@@ -32,6 +32,9 @@
     </link>
     <!-- Left finger -->
+    <!-- Origin Y=0.018 (was 0.04): at q=0 the finger plates (half-width 0.015)
+         nearly meet (~6 mm gap) = CLOSED/gripping; at q=0.04 they open ~8 cm.
+         Previously q=0 left a ~5 cm gap so "closed" never looked closed. -->
     <joint name="gripper_left_joint" type="prismatic">
-      <origin xyz="0 0.04 0" rpy="0 0 0"/>
+      <origin xyz="0 0.018 0" rpy="0 0 0"/>
       <parent link="gripper_base_link"/>
       <child link="gripper_left_link"/>
@@ -64,5 +67,6 @@
       </inertial>
     </link>
-    <!-- Right finger (mirrored).
+    <!-- Right finger (mirrored). Origin Y=-0.018 to match the left finger. -->
+    <!-- ORIGINAL_NOTE:
          URDF <mimic> tag RESTORED: robot_state_publisher reads this to compute
          gripper_right_link TF and MoveIt needs the real URDF joint model.
@@ -78,5 +82,5 @@
          MoveIt's joint-not-found spam is eliminated. -->
     <joint name="gripper_right_joint" type="prismatic">
-      <origin xyz="0 -0.04 0" rpy="0 0 0"/>
+      <origin xyz="0 -0.018 0" rpy="0 0 0"/>
       <parent link="gripper_base_link"/>
       <child link="gripper_right_link"/>
