Commit message: Fix camera optical frames + reshape gripper fingers
- camera.xacro: optical frames rpy="0 0 0" so the gz camera (+X view axis)
  points forward and is upright (was -1.5708 0 -1.5708, which aimed the view
  sideways and made the simulated image ~90 deg off).
- gripper.xacro: fingers are flat plates facing forward, rolled 90 deg about X
  and pushed forward (origin x 0.04) to sit against the front of the base block.

Co-Authored-By: Claude Opus 4.8 (1M context) <noreply@anthropic.com>

File: urdf/components/camera.xacro (robot description, xacro)
@@ -33,14 +33,16 @@
       </inertial>
     </link>
-    <!-- Left camera optical frame -->
+    <!-- Left camera optical frame.
+         Ignition's camera images along the frame +X. rpy="0 0 0" points
+         +X forward (the view direction) and rolls -90 deg about it. -->
     <joint name="camera_left_optical_joint" type="fixed">
-      <origin xyz="0.045 0.0275 0" rpy="-1.5708 0 -1.5708"/>
+      <origin xyz="0.045 0.0275 0" rpy="0 0 0"/>
       <parent link="camera_link"/>
       <child link="camera_left_optical_frame"/>
     </joint>
     <link name="camera_left_optical_frame"/>
-    <!-- Right camera optical frame -->
+    <!-- Right camera optical frame (see left frame note). -->
     <joint name="camera_right_optical_joint" type="fixed">
-      <origin xyz="0.045 -0.0275 0" rpy="-1.5708 0 -1.5708"/>
+      <origin xyz="0.045 -0.0275 0" rpy="0 0 0"/>
       <parent link="camera_link"/>
       <child link="camera_right_optical_frame"/>

File: urdf/components/gripper.xacro (robot description, xacro)
@@ -42,19 +42,19 @@
     <link name="gripper_left_link">
       <visual>
-        <origin xyz="0 0.015 0" rpy="0 0 0"/>
+        <origin xyz="0.04 0 0" rpy="1.5708 0 0"/>
         <geometry>
-          <box size="0.01 0.03 0.04"/>
+          <box size="0.04 0.01 0.03"/>
         </geometry>
         <material name="gripper_dark"/>
       </visual>
       <collision>
-        <origin xyz="0 0.015 0" rpy="0 0 0"/>
+        <origin xyz="0.04 0 0" rpy="1.5708 0 0"/>
         <geometry>
-          <box size="0.01 0.03 0.04"/>
+          <box size="0.04 0.01 0.03"/>
         </geometry>
       </collision>
       <inertial>
         <mass value="0.01"/>
-        <origin xyz="0 0.015 0"/>
+        <origin xyz="0.04 0 0"/>
         <inertia ixx="0.0000005" ixy="0" ixz="0"
                  iyy="0.0000005" iyz="0"
@@ -74,19 +74,19 @@
     <link name="gripper_right_link">
       <visual>
-        <origin xyz="0 -0.015 0" rpy="0 0 0"/>
+        <origin xyz="0.04 0 0" rpy="1.5708 0 0"/>
         <geometry>
-          <box size="0.01 0.03 0.04"/>
+          <box size="0.04 0.01 0.03"/>
         </geometry>
         <material name="gripper_dark"/>
       </visual>
       <collision>
-        <origin xyz="0 -0.015 0" rpy="0 0 0"/>
+        <origin xyz="0.04 0 0" rpy="1.5708 0 0"/>
         <geometry>
-          <box size="0.01 0.03 0.04"/>
+          <box size="0.04 0.01 0.03"/>
         </geometry>
       </collision>
       <inertial>
         <mass value="0.01"/>
-        <origin xyz="0 -0.015 0"/>
+        <origin xyz="0.04 0 0"/>
         <inertia ixx="0.0000005" ixy="0" ixz="0"
                  iyy="0.0000005" iyz="0"

Commit message: fix(urdf): correct camera optical frames to REP-103 (z-forward)
camera_{left,right}_optical_frame had rpy=0 (body x-forward) but serve as the
image/cloud frame_id, while OpenCV reprojectImageTo3D outputs z-forward -> 90deg
geometry error (Phase 0 finding). Added body frames camera_{left,right}_link for
the gz sensors (Ignition looks +X forward); optical frames are now true optical
children (rpy=-pi/2 0 -pi/2). Verified base_link->camera_left_optical_frame = RPY(-90,0,-90).

Co-Authored-By: Claude Opus 4.8 (1M context) <noreply@anthropic.com>

File: urdf/components/camera.xacro (robot description, xacro)
@@ -33,17 +33,31 @@
       </inertial>
     </link>
-    <!-- Left camera optical frame.
-         Ignition's camera images along the frame +X. rpy="0 0 0" points
-         +X forward (the view direction) and rolls -90 deg about it. -->
-    <joint name="camera_left_optical_joint" type="fixed">
+    <!-- Camera BODY frames (REP-103: +X forward). Ignition's camera looks along
+         the +X of the frame the <sensor> is attached to, so the gz sensors mount
+         here to look forward. -->
+    <joint name="camera_left_joint" type="fixed">
       <origin xyz="0.045 0.0275 0" rpy="0 0 0"/>
       <parent link="camera_link"/>
+      <child link="camera_left_link"/>
+    </joint>
+    <link name="camera_left_link"/>
+    <joint name="camera_right_joint" type="fixed">
+      <origin xyz="0.045 -0.0275 0" rpy="0 0 0"/>
+      <parent link="camera_link"/>
+      <child link="camera_right_link"/>
+    </joint>
+    <link name="camera_right_link"/>
+    <!-- True OPTICAL frames (REP-103: +Z forward, +X right, +Y down). These are
+         the frame_id for images / disparity / point clouds, so OpenCV's
+         reprojectImageTo3D output (z-forward) is correctly oriented. -->
+    <joint name="camera_left_optical_joint" type="fixed">
+      <origin xyz="0 0 0" rpy="${-pi/2} 0 ${-pi/2}"/>
+      <parent link="camera_left_link"/>
       <child link="camera_left_optical_frame"/>
     </joint>
     <link name="camera_left_optical_frame"/>
-    <!-- Right camera optical frame (see left frame note). -->
     <joint name="camera_right_optical_joint" type="fixed">
-      <origin xyz="0.045 -0.0275 0" rpy="0 0 0"/>
-      <parent link="camera_link"/>
+      <origin xyz="0 0 0" rpy="${-pi/2} 0 ${-pi/2}"/>
+      <parent link="camera_right_link"/>
       <child link="camera_right_optical_frame"/>
     </joint>
@@ -55,6 +69,7 @@
     <!-- Gazebo Stereo Camera Sensors (simulation only) -->
     <!-- Matches IMX219-83 hardware: 640×360, 30fps, 73° FOV, 60mm baseline -->
-    <!-- LEFT CAMERA -->
-    <gazebo reference="camera_left_optical_frame">
+    <!-- LEFT CAMERA — sensor on the body frame (looks +X forward); images tagged
+         with the optical frame via ignition_frame_id. -->
+    <gazebo reference="camera_left_link">
       <sensor name="stereo_camera_left" type="camera">
         <topic>stereo_camera/left/image_raw</topic>
@@ -91,6 +106,7 @@
       </sensor>
     </gazebo>
-    <!-- RIGHT CAMERA -->
-    <gazebo reference="camera_right_optical_frame">
+    <!-- RIGHT CAMERA — sensor on the body frame (looks +X forward); images tagged
+         with the optical frame via ignition_frame_id. -->
+    <gazebo reference="camera_right_link">
       <sensor name="stereo_camera_right" type="camera">
         <topic>stereo_camera/right/image_raw</topic>

Commit message: chore(audit): cross-4 set stereo camera baseline to 60mm matching IMX219-83
Sim camera y-offsets were +/-0.0275 (55mm) while the file's own comment,
the IMX219-83 spec, and the perception config/static TF all use 60mm.
Sim reprojection (baseline 0.06) now matches the simulated geometry.

Co-Authored-By: Claude Fable 5 <noreply@anthropic.com>
Claude-Session: https://claude.ai/code/session_01Bdt8eBeQJ66FaP4h5R7Gmt

File: urdf/components/camera.xacro (robot description, xacro)
@@ -37,5 +37,5 @@
          here to look forward. -->
     <joint name="camera_left_joint" type="fixed">
-      <origin xyz="0.045 0.0275 0" rpy="0 0 0"/>
+      <origin xyz="0.045 0.03 0" rpy="0 0 0"/>
       <parent link="camera_link"/>
       <child link="camera_left_link"/>
@@ -43,5 +43,5 @@
     <link name="camera_left_link"/>
     <joint name="camera_right_joint" type="fixed">
-      <origin xyz="0.045 -0.0275 0" rpy="0 0 0"/>
+      <origin xyz="0.045 -0.03 0" rpy="0 0 0"/>
       <parent link="camera_link"/>
       <child link="camera_right_link"/>
